File: music_box_pcb/music_box_pcb.kicad_pcb (KiCad board)
At the start: 2 copper layers, 210 x 240 mm, 66 parts

Commit message: LED placement
Parts:
- removed MP1: SLP3-200-100-F, SLP3-200-100-F:BIVAR_SLP3-200-100-F
- D1, D10, D19, D28, D61, D62, D63, D64: footprint LED_SMD:LED_WS2812B_PLCC4_5.0x5.0mm_P3.2mm -> music_box_pcb:LED_SK6812_3535_with_pipe
- D11: renamed from D18; footprint LED_SMD:LED_WS2812B_PLCC4_5.0x5.0mm_P3.2mm -> music_box_pcb:LED_SK6812_3535_with_pipe
- D12: renamed from D26; footprint LED_SMD:LED_WS2812B_PLCC4_5.0x5.0mm_P3.2mm -> music_box_pcb:LED_SK6812_3535_with_pipe
- D13: renamed from D37; footprint LED_SMD:LED_WS2812B_PLCC4_5.0x5.0mm_P3.2mm -> music_box_pcb:LED_SK6812_3535_with_pipe
- D14: renamed from D38; footprint LED_SMD:LED_WS2812B_PLCC4_5.0x5.0mm_P3.2mm -> music_box_pcb:LED_SK6812_3535_with_pipe
- D15: renamed from D39; footprint LED_SMD:LED_WS2812B_PLCC4_5.0x5.0mm_P3.2mm -> music_box_pcb:LED_SK6812_3535_with_pipe
- D16: renamed from D40; footprint LED_SMD:LED_WS2812B_PLCC4_5.0x5.0mm_P3.2mm -> music_box_pcb:LED_SK6812_3535_with_pipe
- D17: renamed from D3; footprint LED_SMD:LED_WS2812B_PLCC4_5.0x5.0mm_P3.2mm -> music_box_pcb:LED_SK6812_3535_with_pipe
- D18: renamed from D11; footprint LED_SMD:LED_WS2812B_PLCC4_5.0x5.0mm_P3.2mm -> music_box_pcb:LED_SK6812_3535_with_pipe
- D2: renamed from D9; footprint LED_SMD:LED_WS2812B_PLCC4_5.0x5.0mm_P3.2mm -> music_box_pcb:LED_SK6812_3535_with_pipe
- D20: renamed from D27; footprint LED_SMD:LED_WS2812B_PLCC4_5.0x5.0mm_P3.2mm -> music_box_pcb:LED_SK6812_3535_with_pipe
- D21: renamed from D41; footprint LED_SMD:LED_WS2812B_PLCC4_5.0x5.0mm_P3.2mm -> music_box_pcb:LED_SK6812_3535_with_pipe
- D22: renamed from D42; footprint LED_SMD:LED_WS2812B_PLCC4_5.0x5.0mm_P3.2mm -> music_box_pcb:LED_SK6812_3535_with_pipe
- D23: renamed from D43; footprint LED_SMD:LED_WS2812B_PLCC4_5.0x5.0mm_P3.2mm -> music_box_pcb:LED_SK6812_3535_with_pipe
- D24: renamed from D44; footprint LED_SMD:LED_WS2812B_PLCC4_5.0x5.0mm_P3.2mm -> music_box_pcb:LED_SK6812_3535_with_pipe
- D25: renamed from D4; footprint LED_SMD:LED_WS2812B_PLCC4_5.0x5.0mm_P3.2mm -> music_box_pcb:LED_SK6812_3535_with_pipe
- D26: renamed from D12; footprint LED_SMD:LED_WS2812B_PLCC4_5.0x5.0mm_P3.2mm -> music_box_pcb:LED_SK6812_3535_with_pipe
- D27: renamed from D20; footprint LED_SMD:LED_WS2812B_PLCC4_5.0x5.0mm_P3.2mm -> music_box_pcb:LED_SK6812_3535_with_pipe
- D29: renamed from D45; footprint LED_SMD:LED_WS2812B_PLCC4_5.0x5.0mm_P3.2mm -> music_box_pcb:LED_SK6812_3535_with_pipe
- D3: renamed from D17; footprint LED_SMD:LED_WS2812B_PLCC4_5.0x5.0mm_P3.2mm -> music_box_pcb:LED_SK6812_3535_with_pipe
- D30: renamed from D46; footprint LED_SMD:LED_WS2812B_PLCC4_5.0x5.0mm_P3.2mm -> music_box_pcb:LED_SK6812_3535_with_pipe
- D31: renamed from D47; footprint LED_SMD:LED_WS2812B_PLCC4_5.0x5.0mm_P3.2mm -> music_box_pcb:LED_SK6812_3535_with_pipe
- D32: renamed from D48; footprint LED_SMD:LED_WS2812B_PLCC4_5.0x5.0mm_P3.2mm -> music_box_pcb:LED_SK6812_3535_with_pipe
- D33: renamed from D5; footprint LED_SMD:LED_WS2812B_PLCC4_5.0x5.0mm_P3.2mm -> music_box_pcb:LED_SK6812_3535_with_pipe
- D34: renamed from D13; footprint LED_SMD:LED_WS2812B_PLCC4_5.0x5.0mm_P3.2mm -> music_box_pcb:LED_SK6812_3535_with_pipe
- D35: renamed from D21; footprint LED_SMD:LED_WS2812B_PLCC4_5.0x5.0mm_P3.2mm -> music_box_pcb:LED_SK6812_3535_with_pipe
- D36: renamed from D29; footprint LED_SMD:LED_WS2812B_PLCC4_5.0x5.0mm_P3.2mm -> music_box_pcb:LED_SK6812_3535_with_pipe
- D37: renamed from D49; footprint LED_SMD:LED_WS2812B_PLCC4_5.0x5.0mm_P3.2mm -> music_box_pcb:LED_SK6812_3535_with_pipe
- D38: renamed from D50; footprint LED_SMD:LED_WS2812B_PLCC4_5.0x5.0mm_P3.2mm -> music_box_pcb:LED_SK6812_3535_with_pipe
- D39: renamed from D51; footprint LED_SMD:LED_WS2812B_PLCC4_5.0x5.0mm_P3.2mm -> music_box_pcb:LED_SK6812_3535_with_pipe
- D4: renamed from D25; footprint LED_SMD:LED_WS2812B_PLCC4_5.0x5.0mm_P3.2mm -> music_box_pcb:LED_SK6812_3535_with_pipe
- D40: renamed from D52; footprint LED_SMD:LED_WS2812B_PLCC4_5.0x5.0mm_P3.2mm -> music_box_pcb:LED_SK6812_3535_with_pipe
- D41: renamed from D6; footprint LED_SMD:LED_WS2812B_PLCC4_5.0x5.0mm_P3.2mm -> music_box_pcb:LED_SK6812_3535_with_pipe
- D42: renamed from D14; footprint LED_SMD:LED_WS2812B_PLCC4_5.0x5.0mm_P3.2mm -> music_box_pcb:LED_SK6812_3535_with_pipe
- D43: renamed from D22; footprint LED_SMD:LED_WS2812B_PLCC4_5.0x5.0mm_P3.2mm -> music_box_pcb:LED_SK6812_3535_with_pipe
- D44: renamed from D30; footprint LED_SMD:LED_WS2812B_PLCC4_5.0x5.0mm_P3.2mm -> music_box_pcb:LED_SK6812_3535_with_pipe
- D45: renamed from D53; footprint LED_SMD:LED_WS2812B_PLCC4_5.0x5.0mm_P3.2mm -> music_box_pcb:LED_SK6812_3535_with_pipe
- D46: renamed from D54; footprint LED_SMD:LED_WS2812B_PLCC4_5.0x5.0mm_P3.2mm -> music_box_pcb:LED_SK6812_3535_with_pipe
- D47: renamed from D55; footprint LED_SMD:LED_WS2812B_PLCC4_5.0x5.0mm_P3.2mm -> music_box_pcb:LED_SK6812_3535_with_pipe
- D48: renamed from D56; footprint LED_SMD:LED_WS2812B_PLCC4_5.0x5.0mm_P3.2mm -> music_box_pcb:LED_SK6812_3535_with_pipe
- D49: renamed from D7; footprint LED_SMD:LED_WS2812B_PLCC4_5.0x5.0mm_P3.2mm -> music_box_pcb:LED_SK6812_3535_with_pipe
- D5: renamed from D33; footprint LED_SMD:LED_WS2812B_PLCC4_5.0x5.0mm_P3.2mm -> music_box_pcb:LED_SK6812_3535_with_pipe
- D50: renamed from D15; footprint LED_SMD:LED_WS2812B_PLCC4_5.0x5.0mm_P3.2mm -> music_box_pcb:LED_SK6812_3535_with_pipe
- D51: renamed from D23; footprint LED_SMD:LED_WS2812B_PLCC4_5.0x5.0mm_P3.2mm -> music_box_pcb:LED_SK6812_3535_with_pipe
- D52: renamed from D31; footprint LED_SMD:LED_WS2812B_PLCC4_5.0x5.0mm_P3.2mm -> music_box_pcb:LED_SK6812_3535_with_pipe
- D53: renamed from D57; footprint LED_SMD:LED_WS2812B_PLCC4_5.0x5.0mm_P3.2mm -> music_box_pcb:LED_SK6812_3535_with_pipe
- D54: renamed from D58; footprint LED_SMD:LED_WS2812B_PLCC4_5.0x5.0mm_P3.2mm -> music_box_pcb:LED_SK6812_3535_with_pipe
- D55: renamed from D59; footprint LED_SMD:LED_WS2812B_PLCC4_5.0x5.0mm_P3.2mm -> music_box_pcb:LED_SK6812_3535_with_pipe
- D56: renamed from D60; footprint LED_SMD:LED_WS2812B_PLCC4_5.0x5.0mm_P3.2mm -> music_box_pcb:LED_SK6812_3535_with_pipe
- D57: renamed from D8; footprint LED_SMD:LED_WS2812B_PLCC4_5.0x5.0mm_P3.2mm -> music_box_pcb:LED_SK6812_3535_with_pipe
- D58: renamed from D16; footprint LED_SMD:LED_WS2812B_PLCC4_5.0x5.0mm_P3.2mm -> music_box_pcb:LED_SK6812_3535_with_pipe
- D59: renamed from D24; footprint LED_SMD:LED_WS2812B_PLCC4_5.0x5.0mm_P3.2mm -> music_box_pcb:LED_SK6812_3535_with_pipe
- D6: renamed from D34; footprint LED_SMD:LED_WS2812B_PLCC4_5.0x5.0mm_P3.2mm -> music_box_pcb:LED_SK6812_3535_with_pipe
- D60: renamed from D32; footprint LED_SMD:LED_WS2812B_PLCC4_5.0x5.0mm_P3.2mm -> music_box_pcb:LED_SK6812_3535_with_pipe
- D7: renamed from D35; footprint LED_SMD:LED_WS2812B_PLCC4_5.0x5.0mm_P3.2mm -> music_box_pcb:LED_SK6812_3535_with_pipe
- D8: renamed from D36; footprint LED_SMD:LED_WS2812B_PLCC4_5.0x5.0mm_P3.2mm -> music_box_pcb:LED_SK6812_3535_with_pipe
- D9: renamed from D2; footprint LED_SMD:LED_WS2812B_PLCC4_5.0x5.0mm_P3.2mm -> music_box_pcb:LED_SK6812_3535_with_pipe
- moved D57 326.1 mm to (407.6, 301.1), turned to 45 degrees
- moved D58 305.1 mm to (407.1, 272.1), turned to 45 degrees
- moved D59 289.1 mm to (406.6, 252.1), turned to 45 degrees
- moved D41 288.2 mm to (353.4, 301.5), turned to -135 degrees
- moved D56 272.5 mm to (378.4, 301.6), turned to 135 degrees
- moved D60 269.8 mm to (406.1, 219.1), turned to 45 degrees
- moved D42 265.0 mm to (353.4, 272.7), turned to -45 degrees
- moved D55 257.7 mm to (378.4, 272.8), turned to 45 degrees
- moved D25 256.8 mm to (299.4, 301.5), turned to -135 degrees
- moved D49 255.9 mm to (378.4, 110.7), turned to 45 degrees
- moved D50 246.8 mm to (378.5, 139.7), turned to 135 degrees
- moved D54 246.4 mm to (378.5, 247.7), turned to 135 degrees
- moved D43 244.9 mm to (353.3, 247.7), turned to -135 degrees
- moved D40 241.3 mm to (324.4, 301.7), turned to 135 degrees
- moved D51 240.6 mm to (378.5, 164.7), turned to 45 degrees
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Connections:
- net Net-(D1-VDD) renamed +5V
- D1 pad 3: Net-(D1-VSS) -> GND
- D10 pad 3: Net-(D10-VSS) -> GND
- D11 pad 2: Net-(D18-DOUT) -> Net-(D11-DOUT)
- D11 pad 3: Net-(D17-VSS) -> GND
- D11 pad 4: Net-(D17-DOUT) -> Net-(D10-DOUT)
- D12 pad 2: Net-(D26-DOUT) -> Net-(D12-DOUT)
- D12 pad 3: Net-(D25-VSS) -> GND
- D12 pad 4: Net-(D25-DOUT) -> Net-(D11-DOUT)
- D13 pad 2: Net-(D37-DOUT) -> Net-(D13-DOUT)
- D13 pad 3: Net-(D33-VSS) -> GND
- D13 pad 4: Net-(D33-DOUT) -> Net-(D12-DOUT)
- D14 pad 2: Net-(D38-DOUT) -> Net-(D14-DOUT)
- D14 pad 3: Net-(D34-VSS) -> GND
- D14 pad 4: Net-(D34-DOUT) -> Net-(D13-DOUT)
- D15 pad 2: Net-(D39-DOUT) -> Net-(D15-DOUT)
- D15 pad 3: Net-(D35-VSS) -> GND
- D15 pad 4: Net-(D35-DOUT) -> Net-(D14-DOUT)
- D16 pad 2: Net-(D40-DOUT) -> Net-(D16-DOUT)
- D16 pad 3: Net-(D36-VSS) -> GND
- D16 pad 4: Net-(D36-DOUT) -> Net-(D15-DOUT)
- D17 pad 2: Net-(D3-DOUT) -> Net-(D17-DOUT)
- D17 pad 3: Net-(D1-VSS) -> GND
- D17 pad 4: Net-(D2-DOUT) -> Net-(D16-DOUT)
- D18 pad 2: Net-(D11-DOUT) -> Net-(D18-DOUT)
- D18 pad 3: Net-(D10-VSS) -> GND
- D18 pad 4: Net-(D10-DOUT) -> Net-(D17-DOUT)
- D19 pad 3: Net-(D17-VSS) -> GND
- D2 pad 2: Net-(D10-DIN) -> Net-(D2-DOUT)
- D2 pad 3: Net-(D10-VSS) -> GND
- D2 pad 4: unconnected-(D9-DIN-Pad4) -> Net-(D1-DOUT)
- D20 pad 2: Net-(D27-DOUT) -> Net-(D20-DOUT)
- D20 pad 3: Net-(D25-VSS) -> GND
- D20 pad 4: Net-(D26-DOUT) -> Net-(D19-DOUT)
- D21 pad 2: Net-(D41-DOUT) -> Net-(D21-DOUT)
- D21 pad 3: Net-(D33-VSS) -> GND
- D21 pad 4: Net-(D37-DOUT) -> Net-(D20-DOUT)
- D22 pad 2: unconnected-(D42-DOUT-Pad2) -> Net-(D22-DOUT)
- D22 pad 3: Net-(D34-VSS) -> GND
- D22 pad 4: Net-(D38-DOUT) -> Net-(D21-DOUT)
- D23 pad 2: Net-(D43-DOUT) -> Net-(D23-DOUT)
- D23 pad 3: Net-(D35-VSS) -> GND
- D23 pad 4: Net-(D39-DOUT) -> Net-(D22-DOUT)
- D24 pad 2: Net-(D44-DOUT) -> Net-(D24-DOUT)
- D24 pad 3: Net-(D36-VSS) -> GND
- D24 pad 4: Net-(D40-DOUT) -> Net-(D23-DOUT)
- D25 pad 2: Net-(D4-DOUT) -> Net-(D25-DOUT)
- D25 pad 3: Net-(D1-VSS) -> GND
- D25 pad 4: Net-(D3-DOUT) -> Net-(D24-DOUT)
- D26 pad 2: Net-(D12-DOUT) -> Net-(D26-DOUT)
- D26 pad 3: Net-(D10-VSS) -> GND
- D26 pad 4: Net-(D11-DOUT) -> Net-(D25-DOUT)
- D27 pad 2: Net-(D20-DOUT) -> Net-(D27-DOUT)
- D27 pad 3: Net-(D17-VSS) -> GND
- D27 pad 4: Net-(D19-DOUT) -> Net-(D26-DOUT)
- D28 pad 3: Net-(D25-VSS) -> GND
- D29 pad 2: Net-(D45-DOUT) -> Net-(D29-DOUT)
- D29 pad 3: Net-(D33-VSS) -> GND
- D29 pad 4: Net-(D41-DOUT) -> Net-(D28-DOUT)
- D3 pad 2: Net-(D17-DOUT) -> Net-(D3-DOUT)
- D3 pad 3: Net-(D17-VSS) -> GND
- D3 pad 4: unconnected-(D17-DIN-Pad4) -> Net-(D2-DOUT)
- D30 pad 2: Net-(D46-DOUT) -> Net-(D30-DOUT)
- D30 pad 3: Net-(D34-VSS) -> GND
- D30 pad 4: unconnected-(D46-DIN-Pad4) -> Net-(D29-DOUT)
- D31 pad 2: Net-(D47-DOUT) -> Net-(D31-DOUT)
- D31 pad 3: Net-(D35-VSS) -> GND
- D31 pad 4: Net-(D43-DOUT) -> Net-(D30-DOUT)
- D32 pad 2: Net-(D48-DOUT) -> Net-(D32-DOUT)
- D32 pad 3: Net-(D36-VSS) -> GND
- D32 pad 4: Net-(D44-DOUT) -> Net-(D31-DOUT)
- D33 pad 2: Net-(D5-DOUT) -> Net-(D33-DOUT)
- D33 pad 3: Net-(D1-VSS) -> GND
- D33 pad 4: Net-(D4-DOUT) -> Net-(D32-DOUT)
- D34 pad 2: Net-(D13-DOUT) -> Net-(D34-DOUT)
- D34 pad 3: Net-(D10-VSS) -> GND
- D34 pad 4: Net-(D12-DOUT) -> Net-(D33-DOUT)
- D35 pad 2: Net-(D21-DOUT) -> Net-(D35-DOUT)
- D35 pad 3: Net-(D17-VSS) -> GND
- D35 pad 4: Net-(D20-DOUT) -> Net-(D34-DOUT)
- D36 pad 2: Net-(D29-DOUT) -> Net-(D36-DOUT)
- D36 pad 3: Net-(D25-VSS) -> GND
- D36 pad 4: Net-(D28-DOUT) -> Net-(D35-DOUT)
- D37 pad 2: Net-(D49-DOUT) -> Net-(D37-DOUT)
- D37 pad 3: Net-(D33-VSS) -> GND
- D37 pad 4: Net-(D45-DOUT) -> Net-(D36-DOUT)
- D38 pad 2: unconnected-(D50-DOUT-Pad2) -> Net-(D38-DOUT)
- D38 pad 3: Net-(D34-VSS) -> GND
- D38 pad 4: Net-(D46-DOUT) -> Net-(D37-DOUT)
- D39 pad 2: Net-(D51-DOUT) -> Net-(D39-DOUT)
- D39 pad 3: Net-(D35-VSS) -> GND
- D39 pad 4: Net-(D47-DOUT) -> Net-(D38-DOUT)
- D4 pad 2: Net-(D25-DOUT) -> Net-(D4-DOUT)
- D4 pad 3: Net-(D25-VSS) -> GND
- D4 pad 4: unconnected-(D25-DIN-Pad4) -> Net-(D3-DOUT)
- D40 pad 2: Net-(D52-DOUT) -> Net-(D40-DOUT)
- D40 pad 3: Net-(D36-VSS) -> GND
- D40 pad 4: Net-(D48-DOUT) -> Net-(D39-DOUT)
- D41 pad 2: Net-(D6-DOUT) -> Net-(D41-DOUT)
- D41 pad 3: Net-(D1-VSS) -> GND
- D41 pad 4: Net-(D5-DOUT) -> Net-(D40-DOUT)
- D42 pad 2: Net-(D14-DOUT) -> Net-(D42-DOUT)
- D42 pad 3: Net-(D10-VSS) -> GND
- D42 pad 4: Net-(D13-DOUT) -> Net-(D41-DOUT)
- D43 pad 2: Net-(D22-DOUT) -> Net-(D43-DOUT)
- D43 pad 3: Net-(D17-VSS) -> GND
- D43 pad 4: Net-(D21-DOUT) -> Net-(D42-DOUT)
- D44 pad 2: Net-(D30-DOUT) -> Net-(D44-DOUT)
- D44 pad 3: Net-(D25-VSS) -> GND
- D44 pad 4: Net-(D29-DOUT) -> Net-(D43-DOUT)
- D45 pad 2: Net-(D53-DOUT) -> Net-(D45-DOUT)
- D45 pad 3: Net-(D33-VSS) -> GND
- D45 pad 4: Net-(D49-DOUT) -> Net-(D44-DOUT)
- D46 pad 2: unconnected-(D54-DOUT-Pad2) -> Net-(D46-DOUT)
- D46 pad 3: Net-(D34-VSS) -> GND
- D46 pad 4: unconnected-(D54-DIN-Pad4) -> Net-(D45-DOUT)
- D47 pad 2: Net-(D55-DOUT) -> Net-(D47-DOUT)
- D47 pad 3: Net-(D35-VSS) -> GND
- D47 pad 4: Net-(D51-DOUT) -> Net-(D46-DOUT)
- D48 pad 2: Net-(D56-DOUT) -> Net-(D48-DOUT)
- D48 pad 3: Net-(D36-VSS) -> GND
- D48 pad 4: Net-(D52-DOUT) -> Net-(D47-DOUT)
- D49 pad 2: Net-(D7-DOUT) -> Net-(D49-DOUT)
- D49 pad 3: Net-(D1-VSS) -> GND
- D49 pad 4: Net-(D6-DOUT) -> Net-(D48-DOUT)
- D5 pad 2: Net-(D33-DOUT) -> Net-(D5-DOUT)
- D5 pad 3: Net-(D33-VSS) -> GND
- D5 pad 4: unconnected-(D33-DIN-Pad4) -> Net-(D4-DOUT)
- D50 pad 2: Net-(D15-DOUT) -> Net-(D50-DOUT)
- D50 pad 3: Net-(D10-VSS) -> GND
- D50 pad 4: Net-(D14-DOUT) -> Net-(D49-DOUT)
- D51 pad 2: Net-(D23-DOUT) -> Net-(D51-DOUT)
- D51 pad 3: Net-(D17-VSS) -> GND
- D51 pad 4: Net-(D22-DOUT) -> Net-(D50-DOUT)
- D52 pad 2: Net-(D31-DOUT) -> Net-(D52-DOUT)
- D52 pad 3: Net-(D25-VSS) -> GND
- D52 pad 4: Net-(D30-DOUT) -> Net-(D51-DOUT)
- D53 pad 2: Net-(D57-DOUT) -> Net-(D53-DOUT)
- D53 pad 3: Net-(D33-VSS) -> GND
- D53 pad 4: Net-(D53-DOUT) -> Net-(D52-DOUT)
- D54 pad 2: unconnected-(D58-DOUT-Pad2) -> Net-(D54-DOUT)
- D54 pad 3: Net-(D34-VSS) -> GND
- D54 pad 4: unconnected-(D58-DIN-Pad4) -> Net-(D53-DOUT)
- D55 pad 2: Net-(D59-DOUT) -> Net-(D55-DOUT)
- D55 pad 3: Net-(D35-VSS) -> GND
- D55 pad 4: Net-(D55-DOUT) -> Net-(D54-DOUT)
- D56 pad 2: Net-(D60-DOUT) -> Net-(D56-DOUT)
- D56 pad 3: Net-(D36-VSS) -> GND
- D56 pad 4: Net-(D56-DOUT) -> Net-(D55-DOUT)
- D57 pad 2: unconnected-(D8-DOUT-Pad2) -> Net-(D57-DOUT)
- D57 pad 3: Net-(D1-VSS) -> GND
- D57 pad 4: Net-(D7-DOUT) -> Net-(D56-DOUT)
- D58 pad 2: unconnected-(D16-DOUT-Pad2) -> Net-(D58-DOUT)
- D58 pad 3: Net-(D10-VSS) -> GND
- D58 pad 4: Net-(D15-DOUT) -> Net-(D57-DOUT)
- D59 pad 2: unconnected-(D24-DOUT-Pad2) -> Net-(D59-DOUT)
- D59 pad 3: Net-(D17-VSS) -> GND
- D59 pad 4: Net-(D23-DOUT) -> Net-(D58-DOUT)
- D6 pad 2: Net-(D34-DOUT) -> Net-(D6-DOUT)
- D6 pad 3: Net-(D34-VSS) -> GND
- D6 pad 4: unconnected-(D34-DIN-Pad4) -> Net-(D5-DOUT)
- D60 pad 2: unconnected-(D32-DOUT-Pad2) -> Net-(D60-DOUT)
- D60 pad 3: Net-(D25-VSS) -> GND
- D60 pad 4: Net-(D31-DOUT) -> Net-(D59-DOUT)
- D61 pad 2: unconnected-(D61-DOUT-Pad2) -> Net-(D61-DOUT)
- D61 pad 3: Net-(D33-VSS) -> GND
- D61 pad 4: Net-(D57-DOUT) -> Net-(D60-DOUT)
- D62 pad 2: unconnected-(D62-DOUT-Pad2) -> Net-(D62-DOUT)
- D62 pad 3: Net-(D34-VSS) -> GND
- D62 pad 4: unconnected-(D62-DIN-Pad4) -> Net-(D61-DOUT)
- D63 pad 2: unconnected-(D63-DOUT-Pad2) -> Net-(D63-DOUT)
- D63 pad 3: Net-(D35-VSS) -> GND
- D63 pad 4: Net-(D59-DOUT) -> Net-(D62-DOUT)
- D64 pad 3: Net-(D36-VSS) -> GND
- D64 pad 4: Net-(D60-DOUT) -> Net-(D63-DOUT)
- D7 pad 2: Net-(D35-DOUT) -> Net-(D7-DOUT)
- D7 pad 3: Net-(D35-VSS) -> GND
- D7 pad 4: unconnected-(D35-DIN-Pad4) -> Net-(D6-DOUT)
- D8 pad 2: Net-(D36-DOUT) -> Net-(D8-DOUT)
- D8 pad 3: Net-(D36-VSS) -> GND
- D8 pad 4: unconnected-(D36-DIN-Pad4) -> Net-(D7-DOUT)
- D9 pad 2: Net-(D2-DOUT) -> Net-(D10-DIN)
- D9 pad 3: Net-(D1-VSS) -> GND
- D9 pad 4: Net-(D1-DOUT) -> Net-(D8-DOUT)
Other:
- outline, holes or cut-outs redrawn

Commit message: update schematic and pcb
Parts:
- moved D61 51.6 mm to (407.5, 193.5), turned to -135 degrees
- moved D64 51.0 mm to (407.4, 110.8), turned to -45 degrees
- moved D62 16.3 mm to (407.4, 164.8), turned to -45 degrees
- moved D63 15.6 mm to (407.4, 139.6), turned to -135 degrees
- moved D59 4.61 mm to (407.4, 247.6), turned to -135 degrees
- moved D60 1.36 mm to (407.4, 218.8), turned to -45 degrees
- moved D58 0.53 mm to (407.3, 272.6), turned to -45 degrees
- moved D57 0.41 mm to (407.5, 301.5), turned to -135 degrees
Connections:
- A1 pad 29: unconnected-(A1-GPIO22-Pad29) -> LED_CTRL
- D1 pad 4: unconnected-(D1-DIN-Pad4) -> LED_CTRL
Routing:
- net Net-(D48-DOUT): track 0.00 -> 49.3 mm
- net Net-(D32-DOUT): track 0.00 -> 45.7 mm
- net Net-(D16-DOUT): track 0.00 -> 41.2 mm
- net Net-(D45-DOUT): track 0.00 -> 31.8 mm
- net Net-(D41-DOUT): track 0.00 -> 31.6 mm
- net Net-(D39-DOUT): track 0.00 -> 31.3 mm
- net Net-(D27-DOUT): track 0.00 -> 31.3 mm
- net Net-(D35-DOUT): track 0.00 -> 31.3 mm
- net Net-(D29-DOUT): track 0.00 -> 30.9 mm
- net Net-(D51-DOUT): track 0.00 -> 30.5 mm
- net Net-(D13-DOUT): track 0.00 -> 30.4 mm
- net Net-(D37-DOUT): track 0.00 -> 30.3 mm
- net Net-(D19-DOUT): track 0.00 -> 30.3 mm
- net Net-(D25-DOUT): track 0.00 -> 30.2 mm
- net Net-(D53-DOUT): track 0.00 -> 30.1 mm
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- added copper zone on F.Cu, net GND

Commit message: update scheamtic/pcb
Parts:
- added C1: 470µF, 16V, Capacitor_SMD:CP_Elec_8x10.5, B.Cu at (310.8, 87.5)
- added C10: 100nF, Capacitor_SMD:C_0603_1608Metric_Pad1.08x0.95mm_HandSolder, F.Cu at (247.5, 259.9)
- added C11: 100nF, Capacitor_SMD:C_0603_1608Metric_Pad1.08x0.95mm_HandSolder, F.Cu at (268.6, 152.0)
- added C12: 100nF, Capacitor_SMD:C_0603_1608Metric_Pad1.08x0.95mm_HandSolder, F.Cu at (270.0, 260.0)
- added C13: 100nF, Capacitor_SMD:C_0603_1608Metric_Pad1.08x0.95mm_HandSolder, F.Cu at (301.9, 152.0)
- added C14: 100nF, Capacitor_SMD:C_0603_1608Metric_Pad1.08x0.95mm_HandSolder, F.Cu at (301.6, 259.5)
- added C15: 100nF, Capacitor_SMD:C_0603_1608Metric_Pad1.08x0.95mm_HandSolder, F.Cu at (323.6, 151.9)
- added C16: 100nF, Capacitor_SMD:C_0603_1608Metric_Pad1.08x0.95mm_HandSolder, F.Cu at (323.1, 259.4)
- added C17: 100nF, Capacitor_SMD:C_0603_1608Metric_Pad1.08x0.95mm_HandSolder, F.Cu at (355.1, 151.9)
- added C18: 100nF, Capacitor_SMD:C_0603_1608Metric_Pad1.08x0.95mm_HandSolder, F.Cu at (354.0, 260.4)
- added C19: 100nF, Capacitor_SMD:C_0603_1608Metric_Pad1.08x0.95mm_HandSolder, F.Cu at (376.4, 152.0)
- added C2: 470µF, 16V, Capacitor_SMD:CP_Elec_8x10.5, B.Cu at (327.3, 87.0)
- added C20: 100nF, Capacitor_SMD:C_0603_1608Metric_Pad1.08x0.95mm_HandSolder, F.Cu at (377.0, 260.4)
- added C21: 100nF, Capacitor_SMD:C_0603_1608Metric_Pad1.08x0.95mm_HandSolder, F.Cu at (408.5, 152.4)
- added C22: 100nF, Capacitor_SMD:C_0603_1608Metric_Pad1.08x0.95mm_HandSolder, F.Cu at (408.0, 259.5)
- added C23: 100pF, Capacitor_SMD:C_0603_1608Metric_Pad1.08x0.95mm_HandSolder, F.Cu at (255.6, 139.5)
- added C24: 100pF, Capacitor_SMD:C_0603_1608Metric_Pad1.08x0.95mm_HandSolder, F.Cu at (256.1, 158.5)
- added C25: 100pF, Capacitor_SMD:C_0603_1608Metric_Pad1.08x0.95mm_HandSolder, F.Cu at (256.1, 243.5)
- added C26: 100pF, Capacitor_SMD:C_0603_1608Metric_Pad1.08x0.95mm_HandSolder, F.Cu at (255.6, 271.0)
- added C3: 470µF, 16V, Capacitor_SMD:CP_Elec_8x10.5, B.Cu at (231.2, 102.0)
- added C4: 470µF, 16V, Capacitor_SMD:CP_Elec_8x10.5, B.Cu at (284.7, 103.0)
- added C5: 470µF, 16V, Capacitor_SMD:CP_Elec_8x10.5, B.Cu at (339.2, 103.0)
- added C6: 470µF, 16V, Capacitor_SMD:CP_Elec_8x10.5, B.Cu at (392.2, 103.0)
- added C7: 100nF, Capacitor_SMD:C_0603_1608Metric_Pad1.08x0.95mm_HandSolder, F.Cu at (212.5, 152.0)
- added C8: 100nF, Capacitor_SMD:C_0603_1608Metric_Pad1.08x0.95mm_HandSolder, F.Cu at (215.0, 259.9)
- added C9: 100nF, Capacitor_SMD:C_0603_1608Metric_Pad1.08x0.95mm_HandSolder, F.Cu at (247.0, 152.0)
- added J1: Conn_01x01_Pin, music_box_pcb:FASTON-2.8, F.Cu at (251.5, 124.0)
- added J10: Conn_01x01_Pin, music_box_pcb:FASTON-2.8, F.Cu at (260.0, 143.5)
- added J11: Conn_01x01_Pin, music_box_pcb:FASTON-2.8, F.Cu at (263.5, 171.6)
- added J12: Conn_01x01_Pin, music_box_pcb:FASTON-2.8, F.Cu at (260.0, 162.5)
- added J13: Conn_01x01_Pin, music_box_pcb:FASTON-2.8, F.Cu at (262.4, 233.1)
- added J14: Conn_01x01_Pin, music_box_pcb:FASTON-2.8, F.Cu at (260.0, 247.5)
- added J15: Conn_01x01_Pin, music_box_pcb:FASTON-2.8, F.Cu at (264.5, 286.0)
- added J16: Conn_01x01_Pin, music_box_pcb:FASTON-2.8, F.Cu at (259.5, 267.1)
- added J17: Conn_01x01_Pin, music_box_pcb:FASTON-2.8, F.Cu at (359.0, 124.5)
- added J18: Conn_01x01_Pin, music_box_pcb:FASTON-2.8, F.Cu at (363.5, 147.0)
- added J19: Conn_01x01_Pin, music_box_pcb:FASTON-2.8, F.Cu at (358.5, 179.5)
- added J2: Conn_01x01_Pin, music_box_pcb:FASTON-2.8, F.Cu at (256.5, 143.5)
- added J20: Conn_01x01_Pin, music_box_pcb:FASTON-2.8, F.Cu at (363.5, 158.6)
- added J21: Conn_01x01_Pin, music_box_pcb:FASTON-2.8, F.Cu at (359.5, 232.5)
- added J22: Conn_01x01_Pin, music_box_pcb:FASTON-2.8, F.Cu at (362.5, 256.0)
- added J23: Conn_01x01_Pin, music_box_pcb:FASTON-2.8, F.Cu at (359.0, 286.5)
- added J24: Conn_01x01_Pin, music_box_pcb:FASTON-2.8, F.Cu at (362.5, 265.5)
- added J25: Conn_01x01_Pin, music_box_pcb:FASTON-2.8, F.Cu at (372.5, 124.5)
- added J26: Conn_01x01_Pin, music_box_pcb:FASTON-2.8, F.Cu at (367.5, 147.0)
- added J27: Conn_01x01_Pin, music_box_pcb:FASTON-2.8, F.Cu at (372.5, 179.0)
- added J28: Conn_01x01_Pin, music_box_pcb:FASTON-2.8, F.Cu at (367.5, 158.6)
- added J29: Conn_01x01_Pin, music_box_pcb:FASTON-2.8, F.Cu at (373.0, 232.5)
- added J3: Conn_01x01_Pin, music_box_pcb:FASTON-2.8, F.Cu at (252.0, 171.6)
- added J30: Conn_01x01_Pin, music_box_pcb:FASTON-2.8, F.Cu at (369.0, 256.0)
- added J31: Conn_01x01_Pin, music_box_pcb:FASTON-2.8, F.Cu at (373.0, 286.0)
- added J32: Conn_01x01_Pin, music_box_pcb:FASTON-2.8, F.Cu at (369.0, 265.5)
- added J33: Conn_01x03_Pin, Connector_JST:JST_XH_B3B-XH-A_1x03_P2.50mm_Vertical, B.Cu at (330.1, 76.0)
- added J34: Conn_01x08_Pin, Connector_JST:JST_XH_B8B-XH-A_1x08_P2.50mm_Vertical, B.Cu at (370.5, 76.0)
- added J35: Conn_01x03_Pin, Connector_JST:JST_XH_B3B-XH-A_1x03_P2.50mm_Vertical, B.Cu at (313.1, 76.0)
- added J4: Conn_01x01_Pin, music_box_pcb:FASTON-2.8, F.Cu at (257.0, 162.5)
- added J5: Conn_01x01_Pin, music_box_pcb:FASTON-2.8, F.Cu at (252.0, 233.0)
- added J6: Conn_01x01_Pin, music_box_pcb:FASTON-2.8, F.Cu at (257.0, 247.5)
- added J7: Conn_01x01_Pin, music_box_pcb:FASTON-2.8, F.Cu at (251.0, 286.5)
- added J8: Conn_01x01_Pin, music_box_pcb:FASTON-2.8, F.Cu at (256.5, 267.2)
- added J9: Conn_01x01_Pin, music_box_pcb:FASTON-2.8, F.Cu at (264.0, 124.0)
- added R1: R, Resistor_SMD:R_0603_1608Metric, F.Cu at (198.7, 110.0)
- added R2: R, Resistor_SMD:R_0603_1608Metric, F.Cu at (198.7, 112.5)
- added R3: 4.7k, Resistor_SMD:R_0603_1608Metric_Pad0.98x0.95mm_HandSolder, F.Cu at (263.0, 91.4)
- added R4: 4.7k, Resistor_SMD:R_0603_1608Metric_Pad0.98x0.95mm_HandSolder, F.Cu at (265.0, 91.4)
- added R5: 4.7k, Resistor_SMD:R_0603_1608Metric_Pad0.98x0.95mm_HandSolder, F.Cu at (267.0, 91.4)
- added R6: 4.7k, Resistor_SMD:R_0603_1608Metric_Pad0.98x0.95mm_HandSolder, F.Cu at (269.1, 91.4)
- added R7: 330, Resistor_SMD:R_0603_1608Metric_Pad0.98x0.95mm_HandSolder, F.Cu at (259.2, 101.3)
- added R8: 330, Resistor_SMD:R_0603_1608Metric_Pad0.98x0.95mm_HandSolder, F.Cu at (300.6, 99.5)
- added R9: 330, Resistor_SMD:R_0603_1608Metric_Pad0.98x0.95mm_HandSolder, F.Cu at (300.6, 96.0)
- A1: footprint Module:RaspberryPi_Pico_Common_Unspecified -> Module:RaspberryPi_Pico_Common_THT; moved to B.Cu
- moved A1 73.8 mm to (237.9, 77.0), turned to -90 degrees
Connections:
- A1 pad 10: unconnected-(A1-GPIO7-Pad10) -> SW_L2
- A1 pad 11: unconnected-(A1-GPIO8-Pad11) -> SW_L3
- A1 pad 12: unconnected-(A1-GPIO9-Pad12) -> SW_L4
- A1 pad 13: Net-(A1-GND-Pad13) -> GND
- A1 pad 14: unconnected-(A1-GPIO10-Pad14) -> Net-(A1-GPIO10)
- A1 pad 15: unconnected-(A1-GPIO11-Pad15) -> Net-(A1-GPIO11)
- A1 pad 16: unconnected-(A1-GPIO12-Pad16) -> Net-(A1-GPIO12)
- A1 pad 18: Net-(A1-GND-Pad13) -> GND
- A1 pad 23: Net-(A1-GND-Pad13) -> GND
- A1 pad 28: Net-(A1-GND-Pad13) -> GND
- A1 pad 29: LED_CTRL -> unconnected-(A1-GPIO22-Pad29)
- A1 pad 3: Net-(A1-GND-Pad13) -> GND
- A1 pad 33: unconnected-(A1-AGND-Pad33) -> GND
- A1 pad 36: unconnected-(A1-3V3-Pad36) -> +3.3V
- A1 pad 38: Net-(A1-GND-Pad13) -> GND
- A1 pad 4: unconnected-(A1-GPIO2-Pad4) -> SW_C1
- A1 pad 5: unconnected-(A1-GPIO3-Pad5) -> SW_C2
- A1 pad 6: unconnected-(A1-GPIO4-Pad6) -> SW_C3
- A1 pad 7: unconnected-(A1-GPIO5-Pad7) -> SW_C4
- A1 pad 8: Net-(A1-GND-Pad13) -> GND
- A1 pad 9: unconnected-(A1-GPIO6-Pad9) -> SW_L1
Routing:
- net SW_C3: track 0.00 -> 157.1 mm, vias 0 -> 2
- net SW_C4: track 0.00 -> 156.0 mm, vias 0 -> 2
- net SW_L1: track 0.00 -> 108.5 mm, vias 0 -> 4
- net GND: track 0.00 -> 53.3 mm, vias 0 -> 35
- net STRIP_1: track 0.00 -> 45.1 mm
- net STRIP_2: track 0.00 -> 27.3 mm
- net Net-(A1-GPIO11): track 0.00 -> 19.8 mm
- net Net-(A1-GPIO12): track 0.00 -> 16.5 mm
- net Net-(D45-DOUT): track 31.8 -> 28.0 mm
- net Net-(D16-DOUT): track 41.2 -> 37.7 mm, vias 0 -> 2
- net Net-(D41-DOUT): track 31.6 -> 28.3 mm
- net Net-(D27-DOUT): track 31.3 -> 28.0 mm
- net Net-(D29-DOUT): track 30.9 -> 28.0 mm
- net Net-(D19-DOUT): track 30.3 -> 27.4 mm
- net Net-(D13-DOUT): track 30.4 -> 27.5 mm
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- added copper zone on F.Cu, net +5V
- added copper zone on B.Cu, net GND
- removed copper zone on F.Cu, net GND
Other:
- outline, holes or cut-outs redrawn
