File: music_box_pcb/led.kicad_sch (KiCad schematic)
At the start: 64 parts

Commit message: update schematic and pcb
Connections:
- net LED_CTRL: now reaches D1.4 (DIN)
Changed lines of the file:
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@@
+	(wire
+		(pts
+			(xy 62.23 38.1) (xy 76.2 38.1)
+		)
+		(stroke
+			(width 0)
+			(type default)
+		)
+	)
 	(wire
 		(pts
@@
 		)
 	)
+	(global_label "LED_CTRL"
+		(shape input)
+		(at 62.23 38.1 180)
+		(fields_autoplaced yes)
+		(effects
+			(font
+				(size 1.27 1.27)
+			)
+			(justify right)
+		)
+		(property "Intersheetrefs" "${INTERSHEET_REFS}"
+			(at 50.2944 38.1 0)
+			(hide yes)
+			(show_name no)
+			(do_not_autoplace no)
+			(effects
+				(font
+					(size 1.27 1.27)
+				)
+				(justify right)
+			)
+		)
+	)

Commit message: update sch and routing
Connections:
- net LED_CTRL renamed SW_LED_CTRL
Changed lines of the file:
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@@
 		)
 	)
-	(global_label "LED_CTRL"
+	(global_label "SW_LED_CTRL"
 		(shape input)
 		(at 62.23 38.1 180)
@@
 		)
 		(property "Intersheetrefs" "${INTERSHEET_REFS}"
-			(at 50.2944 38.1 0)
+			(at 46.6659 38.1 0)
 			(hide yes)
 			(show_name no)
