File: music_box_pcb/music_box_pcb.kicad_sch (KiCad schematic)
At the start: 1 part

Commit message: update schematic and pcb
Connections:
- net LED_CTRL: now reaches A1.29 (GPIO22)
Changed lines of the file:
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@@
 	(generator_version "10.0")
 	(paper "A4")
+	(wire
+		(pts
+			(xy 130.81 87.63) (xy 168.91 87.63)
+		)
+		(stroke
+			(width 0)
+			(type default)
+		)
+	)
+	(wire
+		(pts
+			(xy 168.91 78.74) (xy 184.15 78.74)
+		)
+		(stroke
+			(width 0)
+			(type default)
+		)
+	)
+	(wire
+		(pts
+			(xy 168.91 87.63) (xy 168.91 78.74)
+		)
+		(stroke
+			(width 0)
+			(type default)
+		)
+	)
+	(global_label "LED_CTRL"
+		(shape output)
+		(at 184.15 78.74 0)
+		(fields_autoplaced yes)
+		(effects
+			(font
+				(size 1.27 1.27)
+			)
+			(justify left)
+		)
+		(property "Intersheetrefs" "${INTERSHEET_REFS}"
+			(at 196.0856 78.74 0)
+			(hide yes)
+			(show_name no)
+			(do_not_autoplace no)
+			(effects
+				(font
+					(size 1.27 1.27)
+				)
+				(justify left)
+			)
+		)
+	)
 	(symbol
 		(lib_id "MCU_Module:RaspberryPi_Pico")

Commit message: update scheamtic/pcb
Parts:
- added R7, R8, R9: 330, Resistor_SMD:R_0603_1608Metric_Pad0.98x0.95mm_HandSolder, symbol Device:R
- A1: footprint Module:RaspberryPi_Pico_Common_Unspecified -> Module:RaspberryPi_Pico_Common_THT
Connections:
- net LED_CTRL: now also R7.1; no longer A1.29 (GPIO22)
- net SW_L2: now reaches A1.10 (GPIO7)
- net SW_L3: now reaches A1.11 (GPIO8)
- net SW_L4: now reaches A1.12 (GPIO9)
- net GND: now reaches A1.13 (GND), A1.18 (GND), A1.23 (GND), A1.28 (GND), A1.3 (GND), A1.38 (GND), A1.8 (GND)
- net GND: now also A1.33 (AGND)
- net at A1.14 (GPIO10): now also R7.2
- net at A1.15 (GPIO11): now also R8.2
- net at A1.16 (GPIO12): now also R9.2
- net +3.3V: now reaches A1.36 (3V3)
- net SW_C1: now reaches A1.4 (GPIO2)
- net SW_C2: now reaches A1.5 (GPIO3)
- net SW_C3: now reaches A1.6 (GPIO4)
- net SW_C4: now reaches A1.7 (GPIO5)
- net SW_L1: now reaches A1.9 (GPIO6)
- new net STRIP_1: R8.1
- new net STRIP_2: R9.1

Commit message: update sch and routing
Connections:
- net SW_C1: now also A1.27 (GPIO21); no longer A1.4 (GPIO2)
- net SW_C2: now also A1.26 (GPIO20); no longer A1.5 (GPIO3)
- net SW_C3: now also A1.22 (GPIO17); no longer A1.6 (GPIO4)
- net SW_L1: now also A1.29 (GPIO22); no longer A1.9 (GPIO6)
- net SW_L2: now also A1.25 (GPIO19); no longer A1.10 (GPIO7)
- net SW_L3: now also A1.24 (GPIO18); no longer A1.11 (GPIO8)
- net at A1.14 (GPIO10): no longer R7.2
- net at A1.15 (GPIO11): no longer R8.2
- net at A1.16 (GPIO12): no longer R9.2
- net at A1.19 (GPIO14): now also R9.2
- net at A1.20 (GPIO15): now also R8.2
- net SW_L0: now reaches A1.31 (GPIO26_ADC0)
- net SW_C0: now reaches A1.32 (GPIO27_ADC1)
- net at A1.34 (GPIO28_ADC2): now also R7.2
- net LED_CTRL renamed SW_LED_CTRL
- net SW_C4: no longer names the net of A1.7 (GPIO5)
- net SW_L4: no longer names the net of A1.12 (GPIO9)
Other:
- moved on the sheet: R7, R8, R9
