File: music_box_pcb/button_matrix.kicad_sch (KiCad schematic)
At the start: 65 parts, among them J1 Conn_01x01_Pin, J10 Conn_01x01_Pin, J11 Conn_01x01_Pin, J12 Conn_01x01_Pin, J13 Conn_01x01_Pin, J14 Conn_01x01_Pin, J15 Conn_01x01_Pin, J16 Conn_01x01_Pin, J17 Conn_01x01_Pin, J18 Conn_01x01_Pin, J19 Conn_01x01_Pin, J2 Conn_01x01_Pin, J20 Conn_01x01_Pin, J21 Conn_01x01_Pin, J22 Conn_01x01_Pin, J23 Conn_01x01_Pin, J24 Conn_01x01_Pin, J25 Conn_01x01_Pin, J26 Conn_01x01_Pin, J27 Conn_01x01_Pin, J28 Conn_01x01_Pin, J29 Conn_01x01_Pin, J3 Conn_01x01_Pin, J30 Conn_01x01_Pin, J31 Conn_01x01_Pin, J32 Conn_01x01_Pin, J33 Conn_01x03_Pin, J34 Conn_01x08_Pin, J35 Conn_01x03_Pin, J4 Conn_01x01_Pin, J5 Conn_01x01_Pin, J6 Conn_01x01_Pin, J7 Conn_01x01_Pin, J8 Conn_01x01_Pin, J9 Conn_01x01_Pin

Commit message: update sch and routing
Connections:
- net SW_C4 is gone; now on net SW_C3: J25.1 (Pin_1), J27.1 (Pin_1), J29.1 (Pin_1), J31.1 (Pin_1)
- net SW_L4 is gone; now on net SW_L3: C26.1, J16.1 (Pin_1), J24.1 (Pin_1), J32.1 (Pin_1), J8.1 (Pin_1), R6.2
- net SW_C1: now also J11.1 (Pin_1), J13.1 (Pin_1), J15.1 (Pin_1), J9.1 (Pin_1); no longer J1.1 (Pin_1), J3.1 (Pin_1), J5.1 (Pin_1), J7.1 (Pin_1)
- net SW_C2: now also J17.1 (Pin_1), J19.1 (Pin_1), J21.1 (Pin_1), J23.1 (Pin_1); no longer J11.1 (Pin_1), J13.1 (Pin_1), J15.1 (Pin_1), J9.1 (Pin_1)
- net SW_C3: no longer J17.1 (Pin_1), J19.1 (Pin_1), J21.1 (Pin_1), J23.1 (Pin_1)
- net SW_L1: now also C24.1, J12.1 (Pin_1), J20.1 (Pin_1), J28.1 (Pin_1), J4.1 (Pin_1), R4.2; no longer C23.1, J10.1 (Pin_1), J18.1 (Pin_1), J2.1 (Pin_1), J26.1 (Pin_1), R3.2
- net SW_L2: now also C25.1, J14.1 (Pin_1), J22.1 (Pin_1), J30.1 (Pin_1), J6.1 (Pin_1), R5.2; no longer C24.1, J12.1 (Pin_1), J20.1 (Pin_1), J28.1 (Pin_1), J4.1 (Pin_1), R4.2
- net SW_L3: no longer C25.1, J14.1 (Pin_1), J22.1 (Pin_1), J30.1 (Pin_1), J6.1 (Pin_1), R5.2
- new net SW_C0: J1.1 (Pin_1), J3.1 (Pin_1), J5.1 (Pin_1), J7.1 (Pin_1)
- new net SW_L0: C23.1, J10.1 (Pin_1), J18.1 (Pin_1), J2.1 (Pin_1), J26.1 (Pin_1), R3.2
Changed lines of the file:
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@@
 		)
 	)
-	(global_label "SW_L4"
+	(global_label "SW_L3"
 		(shape output)
 		(at 255.27 67.31 0)
@@
 		)
 	)
-	(global_label "SW_C4"
+	(global_label "SW_C3"
 		(shape input)
 		(at 177.8 17.78 180)
@@
 		)
 	)
+	(global_label "SW_C0"
+		(shape input)
+		(at 36.83 19.05 180)
+		(fields_autoplaced yes)
+		(effects
+			(font
+				(size 1.27 1.27)
+			)
+			(justify right)
+		)
+		(property "Intersheetrefs" "${INTERSHEET_REFS}"
+			(at 27.7368 19.05 0)
+			(hide yes)
+			(show_name no)
+			(do_not_autoplace no)
+			(effects
+				(font
+					(size 1.27 1.27)
+				)
+				(justify right)
+			)
+		)
+	)
+	(global_label "STRIP_1"
+		(shape input)
+		(at 105.41 99.06 0)
+		(fields_autoplaced yes)
+		(effects
+			(font
+				(size 1.27 1.27)
+			)
+			(justify left)
+		)
+		(property "Intersheetrefs" "${INTERSHEET_REFS}"
+			(at 115.8942 99.06 0)
+			(hide yes)
+			(show_name no)
+			(do_not_autoplace no)
+			(effects
+				(font
+					(size 1.27 1.27)
+				)
+				(justify left)
+			)
+		)
+	)
+	(global_label "SW_C2"
+		(shape input)
+		(at 129.54 19.05 180)
+		(fields_autoplaced yes)
+		(effects
+			(font
+				(size 1.27 1.27)
+			)
+			(justify right)
+		)
+		(property "Intersheetrefs" "${INTERSHEET_REFS}"
+			(at 120.4468 19.05 0)
+			(hide yes)
+			(show_name no)
+			(do_not_autoplace no)
+			(effects
+				(font
+					(size 1.27 1.27)
+				)
+				(justify right)
+			)
+		)
+	)
+	(global_label "SW_L2"
+		(shape output)
+		(at 255.27 55.88 0)
+		(fields_autoplaced yes)
+		(effects
+			(font
+				(size 1.27 1.27)
+			)
+			(justify left)
+		)
+		(property "Intersheetrefs" "${INTERSHEET_REFS}"
+			(at 264.1213 55.88 0)
+			(hide yes)
+			(show_name no)
+			(do_not_autoplace no)
+			(effects
+				(font
+					(size 1.27 1.27)
+				)
+				(justify left)
+			)
+		)
+	)
+	(global_label "SW_L1"
+		(shape output)
+		(at 255.27 45.72 0)
+		(fields_autoplaced yes)
+		(effects
+			(font
+				(size 1.27 1.27)
+			)
+			(justify left)
+		)
+		(property "Intersheetrefs" "${INTERSHEET_REFS}"
+			(at 264.1213 45.72 0)
+			(hide yes)
+			(show_name no)
+			(do_not_autoplace no)
+			(effects
+				(font
+					(size 1.27 1.27)
+				)
+				(justify left)
+			)
+		)
+	)
+	(global_label "SW_L0"
+		(shape output)
+		(at 255.27 35.56 0)
+		(fields_autoplaced yes)
+		(effects
+			(font
+				(size 1.27 1.27)
+			)
+			(justify left)
+		)
+		(property "Intersheetrefs" "${INTERSHEET_REFS}"
+			(at 264.1213 35.56 0)
+			(hide yes)
+			(show_name no)
+			(do_not_autoplace no)
+			(effects
+				(font
+					(size 1.27 1.27)
+				)
+				(justify left)
+			)
+		)
+	)
+	(global_label "STRIP_2"
+		(shape input)
+		(at 105.41 116.84 0)
+		(fields_autoplaced yes)
+		(effects
+			(font
+				(size 1.27 1.27)
+			)
+			(justify left)
+		)
+		(property "Intersheetrefs" "${INTERSHEET_REFS}"
+			(at 115.8942 116.84 0)
+			(hide yes)
+			(show_name no)
+			(do_not_autoplace no)
+			(effects
+				(font
+					(size 1.27 1.27)
+				)
+				(justify left)
+			)
+		)
+	)
 	(global_label "SW_C1"
 		(shape input)
-		(at 36.83 19.05 180)
-		(fields_autoplaced yes)
-		(effects
-			(font
-				(size 1.27 1.27)
-			)
-			(justify right)
-		)
-		(property "Intersheetrefs" "${INTERSHEET_REFS}"
-			(at 27.7368 19.05 0)
-			(hide yes)
-			(show_name no)
-			(do_not_autoplace no)
-			(effects
-				(font
-					(size 1.27 1.27)
-				)
-				(justify right)
-			)
-		)
-	)
-	(global_label "STRIP_1"
-		(shape input)
-		(at 105.41 99.06 0)
-		(fields_autoplaced yes)
-		(effects
-			(font
-				(size 1.27 1.27)
-			)
-			(justify left)
-		)
-		(property "Intersheetrefs" "${INTERSHEET_REFS}"
-			(at 115.8942 99.06 0)
-			(hide yes)
-			(show_name no)
-			(do_not_autoplace no)
-			(effects
-				(font
-					(size 1.27 1.27)
-				)
-				(justify left)
-			)
-		)
-	)
-	(global_label "SW_C3"
-		(shape input)
-		(at 129.54 19.05 180)
-		(fields_autoplaced yes)
-		(effects
-			(font
-				(size 1.27 1.27)
-			)
-			(justify right)
-		)
-		(property "Intersheetrefs" "${INTERSHEET_REFS}"
-			(at 120.4468 19.05 0)
-			(hide yes)
-			(show_name no)
-			(do_not_autoplace no)
-			(effects
-				(font
-					(size 1.27 1.27)
-				)
-				(justify right)
-			)
-		)
-	)
-	(global_label "SW_L3"
-		(shape output)
-		(at 255.27 55.88 0)
-		(fields_autoplaced yes)
-		(effects
-			(font
-				(size 1.27 1.27)
-			)
-			(justify left)
-		)
-		(property "Intersheetrefs" "${INTERSHEET_REFS}"
-			(at 264.1213 55.88 0)
-			(hide yes)
-			(show_name no)
-			(do_not_autoplace no)
-			(effects
-				(font
-					(size 1.27 1.27)
-				)
-				(justify left)
-			)
-		)
-	)
-	(global_label "SW_L2"
-		(shape output)
-		(at 255.27 45.72 0)
-		(fields_autoplaced yes)
-		(effects
-			(font
-				(size 1.27 1.27)
-			)
-			(justify left)
-		)
-		(property "Intersheetrefs" "${INTERSHEET_REFS}"
-			(at 264.1213 45.72 0)
-			(hide yes)
-			(show_name no)
-			(do_not_autoplace no)
-			(effects
-				(font
-					(size 1.27 1.27)
-				)
-				(justify left)
-			)
-		)
-	)
-	(global_label "SW_L1"
-		(shape output)
-		(at 255.27 35.56 0)
-		(fields_autoplaced yes)
-		(effects
-			(font
-				(size 1.27 1.27)
-			)
-			(justify left)
-		)
-		(property "Intersheetrefs" "${INTERSHEET_REFS}"
-			(at 264.1213 35.56 0)
-			(hide yes)
-			(show_name no)
-			(do_not_autoplace no)
-			(effects
-				(font
-					(size 1.27 1.27)
-				)
-				(justify left)
-			)
-		)
-	)
-	(global_label "STRIP_2"
-		(shape input)
-		(at 105.41 116.84 0)
-		(fields_autoplaced yes)
-		(effects
-			(font
-				(size 1.27 1.27)
-			)
-			(justify left)
-		)
-		(property "Intersheetrefs" "${INTERSHEET_REFS}"
-			(at 115.8942 116.84 0)
-			(hide yes)
-			(show_name no)
-			(do_not_autoplace no)
-			(effects
-				(font
-					(size 1.27 1.27)
-				)
-				(justify left)
-			)
-		)
-	)
-	(global_label "SW_C2"
-		(shape input)
 		(at 82.55 19.05 180)

Commit message: update schematic/PCB
Parts:
- added C27, C28, C29, C30: 100nF, Capacitor_SMD:C_0603_1608Metric_Pad1.08x0.95mm_HandSolder, symbol Device:C
- added C31: 470µF, 16V, Capacitor_SMD:CP_Elec_8x10.5, symbol Device:C_Polarized
Connections:
- net +5V: now also C27.1, C28.1, C29.1, C30.1, C31.1
- net GND: now also C27.2, C28.2, C29.2, C30.2, C31.2
